Commit message: urdfを修正、エンドエフェクタの座標系が逆になった？

File: mycobot_description/urdf/hma_cobot_with_eef.urdf (robot description, URDF)
Before this commit: robot mycobot_pro_with_gripper, 16 links, 15 joints
Links:
- removed link camera_adaptor
- link gripper_base: geometry collision mesh filename=package://mycobot_description/urdf/f100_gripper/pro_gripper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; visual mesh filename=package://mycobot_description/urdf/f100_gripper/pro_gripper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
- link gripper_left1: geometry collision mesh filename=package://mycobot_description/urdf/f100_gripper/pro_gripper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; visual mesh filename=package://mycobot_description/urdf/f100_gripper/pro_gripper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
- link gripper_left2: geometry collision mesh filename=package://mycobot_description/urdf/f100_gripper/pro_gripper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; visual mesh filename=package://mycobot_description/urdf/f100_gripper/pro_gripper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
- link gripper_left3: geometry collision mesh filename=package://mycobot_description/urdf/f100_gripper/pro_gripper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; visual mesh filename=package://mycobot_description/urdf/f100_gripper/pro_gripper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
- link gripper_right1: geometry collision mesh filename=package://mycobot_description/urdf/f100_gripper/pro_gripper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; visual mesh filename=package://mycobot_description/urdf/f100_gripper/pro_gripper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
- link gripper_right2: geometry collision mesh filename=package://mycobot_description/urdf/f100_gripper/pro_gripper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; visual mesh filename=package://mycobot_description/urdf/f100_gripper/pro_gripper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
- link gripper_right3: geometry collision mesh filename=package://mycobot_description/urdf/f100_gripper/pro_gripper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; visual mesh filename=package://mycobot_description/urdf/f100_gripper/pro_gripper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
Joints:
- removed joint camera_adaptor_link
- removed joint flange_to_gripper
- removed joint gripper_left1
- removed joint gripper_left2
- removed joint gripper_right1
- removed joint gripper_right2
- removed joint gripper_right3
- added joint gripper_base_to_gripper_left2: type revolute, parent gripper_base, child gripper_left2, origin xyz=-0.0445 -0.004 -0.02 rpy=0 0 0, axis 0 0 1, limit lower=-0.8 upper=0.5 effort=1000.0 velocity=0, mimic joint=gripper_controller multiplier=1.0 offset=0
- added joint gripper_base_to_gripper_right2: type revolute, parent gripper_base, child gripper_right2, origin xyz=0.0442 -0.004 -0.02 rpy=0 0 0, axis 0 0 1, limit lower=-0.5 upper=0.8 effort=1000.0 velocity=0, mimic joint=gripper_controller multiplier=-1.0 offset=0
- added joint gripper_base_to_gripper_right3: type revolute, parent gripper_base, child gripper_right3, origin xyz=0.018 0.015 -0.0212 rpy=0 0 0, axis 0 0 1, limit lower=1 upper=0 effort=1000.0 velocity=0, mimic joint=gripper_controller multiplier=-1.0 offset=0
- added joint gripper_left3_to_gripper_left1: type revolute, parent gripper_left3, child gripper_left1, origin xyz=0.01 0.06 0.0 rpy=0 0 0, axis 0 0 1, limit lower=-0.5 upper=0.5 effort=1000.0 velocity=0, mimic joint=gripper_controller multiplier=-1.0 offset=0
- added joint gripper_right3_to_gripper_right1: type revolute, parent gripper_right3, child gripper_right1, origin xyz=-0.01 0.061 0.001 rpy=0 0 0, axis 0 0 1, limit lower=-0.5 upper=0.5 effort=1000.0 velocity=0, mimic joint=gripper_controller multiplier=1.0 offset=0
- added joint link6_to_gripper_base: type fixed, parent link6, child gripper_base, origin xyz=-0.04 -0.01 0.01 rpy=0 -0.7854 1.5708
- joint end_effector_joint: origin xyz=0.1 0.0 0.0 rpy=-1.57 0 -1.57 -> xyz=-0.09 0 0 rpy=-1.57 0.785 -1.57; parent camera_adaptor -> link6
- joint gripper_controller: limit lower=-0.7 upper=0.3 effort=1000.0 velocity=0 -> lower=0 upper=1 effort=1000.0 velocity=0; origin xyz=-0.018 0.016 0 rpy=0 0 0 -> xyz=-0.018 0.016 -0.02 rpy=0 0 0
- joint joint6: origin xyz=-0.07586 0 0 rpy=-1.57080 0 0  -> xyz=-0.07586 0 0 rpy=-1.7 0 0 

File: mycobot_description/urdf/hma_cobot_with_eef.xacro (robot description, xacro)
@@ -4,12 +4,14 @@
   <xacro:include filename="$(find mycobot_description)/urdf/mycobot_pro_600/mycobot_pro_600.urdf" />
   <!-- Include camera_attachment URDF -->
-  <xacro:include filename="$(find mycobot_description)/urdf/camera_attachments/camera_attachment.urdf" />
+  <xacro:include filename="$(find mycobot_description)/urdf/f100_gripper/pro_force_gripper.urdf" />
+  <!-- Include camera_attachment URDF -->
+  <!-- <xacro:include filename="$(find mycobot_description)/urdf/camera_attachments/camera_attachment.urdf" /> -->
   <!-- Include Adaptive Gripper URDF -->
-  <xacro:include filename="$(find mycobot_description)/urdf/pro_adaptive_gripper/mycobot_pro_adaptive_gripper.urdf" />
-  <joint name="flange_to_gripper" type="fixed">
+  <!-- <xacro:include filename="$(find mycobot_description)/urdf/pro_adaptive_gripper/mycobot_pro_adaptive_gripper.urdf" /> -->
+  <!-- <joint name="flange_to_gripper" type="fixed">
     <parent link="camera_adaptor"/>
     <child link="gripper_base"/>
     <origin xyz="0.06 -0.007 0" rpy="-1.57 1.57 3.14"/>
-  </joint>
+  </joint> -->
   <!--extension for eef-->
   <link name="end_effector_link">
@@ -22,9 +24,9 @@
   </link>
   <joint name="end_effector_joint" type="fixed">
-    <parent link="camera_adaptor"/>
+    <parent link="link6"/>
     <child link="end_effector_link"/>
     <!--origin xyz="0.1 0.0 0.0" rpy="0 1.57 1.57"/> -->
     <!--origin xyz="0.1 0.0 0.0" rpy="3.14 -1.57 1.57"/-->
-    <origin xyz="0.1 0.0 0.0" rpy="-1.57 0 -1.57"/>
+    <origin xyz="-0.09 0 0" rpy="-1.57 0 -1.57"/>
   </joint>
 </robot>

Commit message: urdfのエンドエフェクタの向きを修正

File: mycobot_description/urdf/hma_cobot_with_eef.urdf (robot description, URDF)
Before this commit: robot mycobot_pro_with_gripper, 15 links, 14 joints
Joints:
- joint end_effector_joint: origin xyz=-0.09 0 0 rpy=-1.57 0.785 -1.57 -> xyz=-0.09 0 0 rpy=2.355 3.14 0.0

Commit message: xacro修正

File: mycobot_description/urdf/hma_cobot_with_eef.urdf (robot description, URDF)
Before this commit: robot mycobot_pro_with_gripper, 15 links, 14 joints
Joints:
- joint joint6: origin xyz=-0.07586 0 0 rpy=-1.7 0 0  -> xyz=-0.07586 0 0 rpy=-1.7 0 0

File: mycobot_description/urdf/hma_cobot_with_eef.xacro (robot description, xacro)
@@ -28,5 +28,5 @@
     <!--origin xyz="0.1 0.0 0.0" rpy="0 1.57 1.57"/> -->
     <!--origin xyz="0.1 0.0 0.0" rpy="3.14 -1.57 1.57"/-->
-    <origin xyz="-0.09 0 0" rpy="-1.57 0 -1.57"/>
+    <origin rpy="2.355 3.14 0.0" xyz="-0.09 0 0"/>
   </joint>
 </robot>

File: mycobot_description/urdf/mycobot_pro_600/mycobot_pro_600.urdf (robot description, URDF)
Before this commit: robot firefighter, 7 links, 6 joints
Joints:
- joint joint6: origin xyz=-0.07586 0 0 rpy=-1.57080 0 0  -> xyz=-0.07586 0 0 rpy=-1.7 0 0
